File: ReallyTuffKinematic GPS PCB/ReallyTuffKinematic GPS.kicad_sch (KiCad schematic)
At the start: 0 parts

Commit message: sync
Parts:
- added BUZZER2: MLT-5020, easyeda2kicad:BUZ-SMD_L5.0-W5.5-P4.60, symbol easyeda2kicad:MLT-5020
- added C10, C4, C5, C6: 4.7uF, Capacitor_SMD:C_0603_1608Metric, symbol Device:C
- added C11, C12, C13, C14, C16, C17, C18, C19, C20, C21, C22, C23, C24, C3: 100nF, Capacitor_SMD:C_0603_1608Metric, symbol Device:C
- added C15: 10uF, Capacitor_SMD:C_0805_2012Metric, symbol Device:C
- added C25: 10uF, Capacitor_SMD:C_0603_1608Metric, symbol Device:C
- added C26: 1uF, Capacitor_SMD:C_0603_1608Metric, symbol Device:C
- added C7, C8: 15pF, Capacitor_SMD:C_0603_1608Metric, symbol Device:C
- added C9: 1nF, Capacitor_SMD:C_0603_1608Metric, symbol Device:C
- added FLASH1: W25Q128JVS, Package_SO:SOIC-8_5.3x5.3mm_P1.27mm, symbol Memory_Flash:W25Q128JVS
- added J1: Conn_01x05_Pin, symbol Connector:Conn_01x05_Pin
- added J2: Conn_01x06_Pin, symbol Connector:Conn_01x06_Pin
- added L1: 3.3uH, Inductor_SMD:L_1210_3225Metric, symbol Device:L
- added R11, R12, R9: 10k, Resistor_SMD:R_0603_1608Metric, symbol Device:R
- added R27: 100, Resistor_SMD:R_0603_1608Metric, symbol Device:R
- added R3, R7, R8: 1k, Resistor_SMD:R_0603_1608Metric, symbol Device:R
- added R6: 33, Resistor_SMD:R_0603_1608Metric, symbol Device:R
- added RP2350: RP2350A, Package_DFN_QFN:QFN-60-1EP_7x7mm_P0.4mm_EP3.4x3.4mm, symbol MCU_RaspberryPi:RP2350A
- added SW2, SW3: SKRPACE010, easyeda2kicad:KEY-SMD_4P-L4.2-W3.2-P2.20-LS4.6, symbol easyeda2kicad:SKRPACE010
- added U1: ESP32-C3-MINI-1-N4, easyeda2kicad:WIFIM-SMD_ESP32-C3-MINI-1, symbol easyeda2kicad:ESP32-C3-MINI-1-N4
- added X1: X322512MSB4SI, easyeda2kicad:CRYSTAL-SMD_4P-L3.2-W2.5-BL, symbol easyeda2kicad:X322512MSB4SI
Connections:
- new net: C4.2, R6.1, RP2350.46 (VREG_AVDD)
- new net: BUZZER2.1 (+), R27.2
- new net: R8.2, SW2.3
- new net: J2.4 (Pin_4), U1.23 (IO9)
- new net: C7.2, R7.1, X1.3 (OSC2)
- new net: R3.2, SW3.1
- new net: L1.2, RP2350.48 (VREG_LX)
- new net: C25.1, U1.3 (3V3)
- new net +1V1: C10.1, C11.1, C12.1, C13.1, C6.2, L1.1, RP2350.23 (DVDD), RP2350.39 (DVDD), RP2350.50 (VREG_FB), RP2350.6 (DVDD)
- new net +3.3V: C14.1, C15.1, C16.1, C17.1, C18.1, C19.1, C20.1, C21.1, C22.1, C23.1, C24.1, C25.2, C3.1, C5.1, FLASH1.8 (VCC), J1.1 (Pin_1), J2.6 (Pin_6), R11.1, R12.1, R6.2, R9.1, RP2350.1 (IOVDD), RP2350.11 (IOVDD), RP2350.20 (IOVDD), RP2350.30 (IOVDD), RP2350.38 (IOVDD), RP2350.44 (ADC_AVDD), RP2350.45 (IOVDD), RP2350.49 (VREG_VIN), RP2350.53 (USB_OTP_VDD), RP2350.54 (QSPI_IOVDD)
- new net GND: BUZZER2.2 (-), C10.2, C11.2, C12.2, C13.2, C14.2, C15.2, C16.2, C17.2, C18.2, C19.2, C20.2, C21.2, C22.2, C23.2, C24.2, C26.1, C3.2, C4.1, C5.2, C6.1, C7.1, C8.1, C9.2, FLASH1.4 (GND), J1.2 (Pin_2), J2.5 (Pin_5), R11.2, R12.2, R8.1, RP2350.47 (VREG_PGND), RP2350.61 (GND), SW3.4, U1.1 (GND), U1.11 (GND), U1.14 (GND), U1.2 (GND), U1.22 (IO8), U1.36 (GND), U1.37 (GND), U1.38 (GND), U1.39 (GND), U1.40 (GND), U1.41 (GND), U1.42 (GND), U1.43 (GND), U1.44 (GND), U1.45 (GND), U1.46 (GND), U1.47 (GND), U1.48 (GND), U1.49 (GND), U1.5 (IO2), U1.50 (GND), U1.51 (GND), U1.52 (GND), U1.53 (GND), X1.2 (GND), X1.4 (GND)
- new net RP2350_GPIO_0: J2.2 (Pin_2), RP2350.2 (GPIO0), U1.30 (RXD0)
- new net RP2350_GPIO_1: J2.1 (Pin_1), RP2350.3 (GPIO1), U1.31 (TXD0)
- new net RP2350_GPIO_10: RP2350.14 (GPIO10)
- new net RP2350_GPIO_11: RP2350.15 (GPIO11)
- new net RP2350_GPIO_12: RP2350.16 (GPIO12)
- new net RP2350_GPIO_13: RP2350.17 (GPIO13)
- new net RP2350_GPIO_14: RP2350.18 (GPIO14)
- new net RP2350_GPIO_15: RP2350.19 (GPIO15)
- new net RP2350_GPIO_16: RP2350.27 (GPIO16)
- new net RP2350_GPIO_17: RP2350.28 (GPIO17)
- new net RP2350_GPIO_18: RP2350.29 (GPIO18)
- new net RP2350_GPIO_19: RP2350.31 (GPIO19)
- new net RP2350_GPIO_2: C26.2, J2.3 (Pin_3), R9.2, RP2350.4 (GPIO2), U1.8 (EN)
- new net RP2350_GPIO_20: RP2350.32 (GPIO20)
- new net RP2350_GPIO_21: RP2350.33 (GPIO21)
- new net RP2350_GPIO_22: R27.1, RP2350.34 (GPIO22)
- new net RP2350_GPIO_23: RP2350.35 (GPIO23)
- new net RP2350_GPIO_24: RP2350.36 (GPIO24)
- new net RP2350_GPIO_25: RP2350.37 (GPIO25)
- new net RP2350_GPIO_26_ADC: RP2350.40 (GPIO26/ADC0)
- new net RP2350_GPIO_27_ADC: RP2350.41 (GPIO27/ADC1)
- new net RP2350_GPIO_28_ADC: RP2350.42 (GPIO28/ADC2)
- new net RP2350_GPIO_29_ADC: RP2350.43 (GPIO29/ADC3)
- new net RP2350_GPIO_3: RP2350.5 (GPIO3)
- new net RP2350_GPIO_4: RP2350.7 (GPIO4)
- new net RP2350_GPIO_5: RP2350.8 (GPIO5)
- new net RP2350_GPIO_6: RP2350.9 (GPIO6)
- new net RP2350_GPIO_7: RP2350.10 (GPIO7)
- new net RP2350_GPIO_8: RP2350.12 (GPIO8)
- new net RP2350_GPIO_9: RP2350.13 (GPIO9)
- new net RP2350_QSPI_SCLK: FLASH1.6 (CLK), RP2350.56 (QSPI_SCLK)
- new net RP2350_QSPI_SD0: FLASH1.5 (DI/IO_{0}), RP2350.57 (QSPI_SD0)
- new net RP2350_QSPI_SD1: FLASH1.2 (DO/IO_{1}), RP2350.59 (QSPI_SD1)
- new net RP2350_QSPI_SD2: FLASH1.3 (~{WP}/IO_{2}), RP2350.58 (QSPI_SD2)
- new net RP2350_QSPI_SD3: FLASH1.7 (~{HOLD}/~{RESET}/IO_{3}), RP2350.55 (QSPI_SD3)
- new net RP2350_QSPI_SS: FLASH1.1 (~{CS}), R3.1, RP2350.60 (~{QSPI_SS})
- new net RP2350_RUN: C9.1, J1.5 (Pin_5), RP2350.26 (RUN), SW2.1
- new net RP2350_SWCLK: J1.3 (Pin_3), RP2350.24 (SWCLK)
- new net RP2350_SWDIO: J1.4 (Pin_4), RP2350.25 (SWDIO)
- new net RP2350_XIN: C8.2, RP2350.21 (XIN), X1.1 (OSC1)
- new net RP2350_XOUT: R7.2, RP2350.22 (XOUT)
- no-connect marks 0 -> 21
Other:
- note added: "1.1V DECOUPLING"
- note added: "3.3V DECOUPLING"
- note added: "BUZZ"
- note added: "ESP32"
- note added: "FLASH RAM"
- note added: "RP2350"
- note added: "RP2350 CRYSTAL"
- note added: "RP2350 DEBUG"
